Commit message: update Motor_Manger with test

File: pi3hat_hw_interface/urdf/test_int.urdf.xacro (robot description, xacro)
@@ -10,4 +10,22 @@
             <param name="I_saturation" >10.0</param>
         </hardware>
+        <joint name="joint1">
+            <command_interface name="position">
+            <param name="min">-1</param>
+            <param name="max">1</param>
+            </command_interface>
+            <state_interface name="position"/>
+            <param name="ID">2</param>
+            <param name="BUS">1</param>
+        </joint>
+         <joint name="joint2">
+            <command_interface name="position">
+            <param name="min">-1</param>
+            <param name="max">1</param>
+            </command_interface>
+            <state_interface name="position"/>
+            <param name="ID">1</param>
+            <param name="BUS">1</param>
+        </joint>
     </ros2_control>
 </robot>

Commit message: first day debug with real hw

File: pi3hat_hw_interface/urdf/test_int.urdf.xacro (robot description, xacro)
@@ -6,10 +6,4 @@
         </hardware>
         <joint name="joint1">
-            <param name="id">2</param>
-            <param name="bus">1</param>
-            <param name="motor_transmission"> 1.0</param>
-            <param name="sec_enc_transmission"> 0.0</param>
-        </joint>
-         <joint name="joint2">
             <param name="id">1</param>
             <param name="bus">1</param>

Commit message: advance in hardware, still comm prob

File: pi3hat_hw_interface/urdf/test_int.urdf.xacro (robot description, xacro)
@@ -6,4 +6,10 @@
         </hardware>
         <joint name="joint1">
+            <param name="id">4</param>
+            <param name="bus">1</param>
+            <param name="motor_transmission"> 1.0</param>
+            <param name="sec_enc_transmission"> 0.0</param>
+        </joint>
+        <joint name="joint2">
             <param name="id">1</param>
             <param name="bus">1</param>

Commit message: set resending false to increased performance

File: pi3hat_hw_interface/urdf/test_int.urdf.xacro (robot description, xacro)
@@ -5,5 +5,5 @@
             <plugin>pi3hat_hw_interface/MoteusPi3Hat_Interface</plugin>
         </hardware>
-        <joint name="joint1">
+         <joint name="joint1">
             <param name="id">2</param>
             <param name="bus">1</param>
@@ -12,4 +12,16 @@
         </joint>
         <joint name="joint2">
+            <param name="id">1</param>
+            <param name="bus">1</param>
+            <param name="motor_transmission"> 1.0</param>
+            <param name="sec_enc_transmission"> 0.0</param>
+        </joint>
+        <joint name="joint3">
+            <param name="id">3</param>
+            <param name="bus">1</param>
+            <param name="motor_transmission"> 1.0</param>
+            <param name="sec_enc_transmission"> 0.0</param>
+        </joint>
+        <joint name="joint4">
             <param name="id">4</param>
             <param name="bus">1</param>

Commit message: fixed bug in command and state interaces, test beg

File: pi3hat_hw_interface/urdf/test_int.urdf.xacro (robot description, xacro)
@@ -5,5 +5,5 @@
             <plugin>pi3hat_hw_interface/MoteusPi3Hat_Interface</plugin>
         </hardware>
-         <joint name="joint1">
+         <!-- <joint name="joint1">
             <param name="id">2</param>
             <param name="bus">1</param>
@@ -18,10 +18,10 @@
         </joint>
         <joint name="joint3">
-            <param name="id">5</param>
+            <param name="id">3</param>
             <param name="bus">1</param>
             <param name="motor_transmission"> 1.0</param>
             <param name="sec_enc_transmission"> 0.0</param>
-        </joint>
-        <joint name="joint4">
+        </joint> -->
+        <joint name="joint">
             <param name="id">4</param>
             <param name="bus">1</param>

Commit message: add second encoder counter and offset

File: pi3hat_hw_interface/urdf/test_int.urdf.xacro (robot description, xacro)
@@ -4,10 +4,10 @@
         <hardware>
             <plugin>pi3hat_hw_interface/MoteusPi3Hat_Interface</plugin>
-            <param name="main_timeout">100</param>
+            <param name="main_timeout">20000</param>
             <param name="can_timeout">20000</param>
             <param name="rcv_timeout">20000</param>
             <param name="attitude">0</param>
         </hardware>
-         <!-- <joint name="joint1">
+         <!-- <joint name="joint3">
             <param name="id">2</param>
             <param name="bus">1</param>
@@ -20,15 +20,15 @@
             <param name="motor_transmission"> 1.0</param>
             <param name="sec_enc_transmission"> 0.0</param>
+        </joint>  -->
+        <joint name="jnt_b9_1Hz_trq4_c2">
+            <param name="id">1</param>
+            <param name="bus">2</param>
+            <param name="motor_transmission"> 9.0</param>
+            <param name="sec_enc_transmission"> 0.0</param>
         </joint>
-        <joint name="joint3">
-            <param name="id">3</param>
+        <joint name="jnt_b9_1Hz_trq4_c3">
+            <param name="id">2</param>
             <param name="bus">1</param>
-            <param name="motor_transmission"> 1.0</param>
-            <param name="sec_enc_transmission"> 0.0</param>
-        </joint> -->
-        <joint name="joint">
-            <param name="id">4</param>
-            <param name="bus">1</param>
-            <param name="motor_transmission"> 1.0</param>
+            <param name="motor_transmission"> 9.0</param>
             <param name="sec_enc_transmission"> 0.0</param>
         </joint>

Commit message: fix sec enc bug, however need more test

File: pi3hat_hw_interface/urdf/test_int.urdf.xacro (robot description, xacro)
@@ -21,5 +21,5 @@
             <param name="sec_enc_transmission"> 0.0</param>
         </joint>  -->
-        <joint name="jnt_b9_1Hz_trq4_c2">
+        <!-- <joint name="jnt_b9_1Hz_trq4_c2">
             <param name="id">1</param>
             <param name="bus">2</param>
@@ -32,4 +32,10 @@
             <param name="motor_transmission"> 9.0</param>
             <param name="sec_enc_transmission"> 0.0</param>
+        </joint> -->
+        <joint name="joint">
+            <param name="id">1</param>
+            <param name="bus">1</param>
+            <param name="motor_transmission">9.0</param>
+            <param name="sec_enc_transmission">3.0</param>
         </joint>
     </ros2_control>

Commit message: fix cycle time and radiant msr&cmd

File: pi3hat_hw_interface/urdf/test_int.urdf.xacro (robot description, xacro)
@@ -4,7 +4,7 @@
         <hardware>
             <plugin>pi3hat_hw_interface/MoteusPi3Hat_Interface</plugin>
-            <param name="main_timeout">20000</param>
-            <param name="can_timeout">20000</param>
-            <param name="rcv_timeout">20000</param>
+            <param name="main_timeout">1500000</param>
+            <param name="can_timeout">90000</param>
+            <param name="rcv_timeout">90000</param>
             <param name="attitude">0</param>
         </hardware>
@@ -33,9 +33,27 @@
             <param name="sec_enc_transmission"> 0.0</param>
         </joint> -->
-        <joint name="joint">
+        <!-- <joint name="joint4">
+            <param name="id">5</param>
+            <param name="bus">1</param>
+            <param name="motor_transmission">9.0</param>
+            <param name="sec_enc_transmission">0.0</param>
+        </joint>
+        <joint name="joint1">
             <param name="id">1</param>
             <param name="bus">1</param>
             <param name="motor_transmission">9.0</param>
-            <param name="sec_enc_transmission">3.0</param>
+            <param name="sec_enc_transmission">0.0</param>
+        </joint>
+        <joint name="joint2">
+            <param name="id">2</param>
+            <param name="bus">1</param>
+            <param name="motor_transmission">9.0</param>
+            <param name="sec_enc_transmission">0.0</param>
+        </joint> -->
+        <joint name="joint">
+            <param name="id">4</param>
+            <param name="bus">1</param>
+            <param name="motor_transmission">1.0</param>
+            <param name="sec_enc_transmission">0.0</param>
         </joint>
     </ros2_control>

Commit message: update current and sec enc

File: pi3hat_hw_interface/urdf/test_int.urdf.xacro (robot description, xacro)
@@ -1,59 +1,23 @@
 <?xml version="1.0" ?>
-<robot name="solo"  xmlns:xacro="http://ros.org/wiki/xacro">
+<robot name="softleg_cart"  xmlns:xacro="http://ros.org/wiki/xacro">
     <ros2_control name="MoteusPi3Hat_Interface" type="system">
         <hardware>
             <plugin>pi3hat_hw_interface/MoteusPi3Hat_Interface</plugin>
-            <param name="main_timeout">1500000</param>
-            <param name="can_timeout">90000</param>
-            <param name="rcv_timeout">90000</param>
+            <param name="main_timeout">400000</param>
+            <param name="can_timeout">20000</param>
+            <param name="rcv_timeout">20000</param>
             <param name="attitude">0</param>
         </hardware>
-         <!-- <joint name="joint3">
-            <param name="id">2</param>
-            <param name="bus">1</param>
-            <param name="motor_transmission"> 1.0</param>
-            <param name="sec_enc_transmission"> 0.0</param>
+        <joint name="joint1"> <!-- hip -->
+            <param name="id">1</param>
+            <param name="bus">2</param>
+            <param name="motor_transmission">9.0</param> <!-- trasmissione primo motore link-->
+            <param name="sec_enc_transmission">2.96</param> <!-- trasmissione secondo motore2enc-->
         </joint>
         <joint name="joint2">
-            <param name="id">1</param>
-            <param name="bus">1</param>
-            <param name="motor_transmission"> 1.0</param>
-            <param name="sec_enc_transmission"> 0.0</param>
-        </joint>  -->
-        <!-- <joint name="jnt_b9_1Hz_trq4_c2">
-            <param name="id">1</param>
-            <param name="bus">2</param>
-            <param name="motor_transmission"> 9.0</param>
-            <param name="sec_enc_transmission"> 0.0</param>
-        </joint>
-        <joint name="jnt_b9_1Hz_trq4_c3">
-            <param name="id">2</param>
-            <param name="bus">1</param>
-            <param name="motor_transmission"> 9.0</param>
-            <param name="sec_enc_transmission"> 0.0</param>
-        </joint> -->
-        <!-- <joint name="joint4">
-            <param name="id">5</param>
-            <param name="bus">1</param>
+           <param name="id">2</param>
+            <param name="bus">3</param>
             <param name="motor_transmission">9.0</param>
-            <param name="sec_enc_transmission">0.0</param>
-        </joint>
-        <joint name="joint1">
-            <param name="id">1</param>
-            <param name="bus">1</param>
-            <param name="motor_transmission">9.0</param>
-            <param name="sec_enc_transmission">0.0</param>
-        </joint>
-        <joint name="joint2">
-            <param name="id">2</param>
-            <param name="bus">1</param>
-            <param name="motor_transmission">9.0</param>
-            <param name="sec_enc_transmission">0.0</param>
-        </joint> -->
-        <joint name="joint">
-            <param name="id">4</param>
-            <param name="bus">1</param>
-            <param name="motor_transmission">1.0</param>
-            <param name="sec_enc_transmission">0.0</param>
+            <param name="sec_enc_transmission">2.87</param>
         </joint>
     </ros2_control>

Commit message: Fix imu problem and adapt frame to our usage

File: pi3hat_hw_interface/urdf/test_int.urdf.xacro (robot description, xacro)
@@ -7,5 +7,5 @@
             <param name="can_timeout">20000</param>
             <param name="rcv_timeout">20000</param>
-            <param name="attitude">0</param>
+            <param name="attitude">1</param>
             <param name="b2imu_pos_x">0</param>
             <param name="b2imu_pos_y">0</param>
@@ -13,18 +13,7 @@
             <param name="b2imu_roll">0</param>
             <param name="b2imu_pitch">0</param>
-            <param name="b2imu_yaw">0</param>
+            <param name="b2imu_yaw">90.0</param>
+            <param name="acc_correction">0</param>
         </hardware>
-        <joint name="joint1"> <!-- hip -->
-            <param name="id">1</param>
-            <param name="bus">2</param>
-            <param name="motor_transmission">9.0</param> <!-- trasmissione primo motore link-->
-            <param name="sec_enc_transmission">2.96</param> <!-- trasmissione secondo motore2enc-->
-        </joint>
-        <joint name="joint2">
-           <param name="id">2</param>
-            <param name="bus">3</param>
-            <param name="motor_transmission">9.0</param>
-            <param name="sec_enc_transmission">2.87</param>
-        </joint>
     </ros2_control>
 </robot>

Commit message: add joint limit, offset and update launch

File: pi3hat_hw_interface/urdf/test_int.urdf.xacro (robot description, xacro)
@@ -16,4 +16,108 @@
             <param name="acc_correction">0</param>
         </hardware>
+        <joint name="RF_HFE">
+            <param name="id">3</param>
+            <param name="bus">4</param>
+            <param name="motor_transmission">9.0</param>
+            <param name="sec_enc_transmission">0.0</param>
+            <param name="KP">0.0</param>
+            <param name="KD">0.0</param>
+            <param name="KI">0.0</param>
+            <param name="i_limit">0.0</param>
+            <param name="p_lim_max">0.0</param>
+            <param name="p_lim_min">0.0</param>
+            <param name="p_offset">0.0</param>
+        </joint>
+        <joint name="RF_KFE"> <!-- hip -->
+            <param name="id">4</param>
+            <param name="bus">4</param>
+            <param name="motor_transmission">9.0</param> <!-- trasmissione primo motore link-->
+            <param name="sec_enc_transmission">0.0</param> <!-- trasmissione secondo motore2enc-->
+            <param name="KP">0.0</param>
+            <param name="KD">0.0</param>
+            <param name="KI">0.0</param>
+            <param name="i_limit">0.0</param>
+            <param name="p_lim_max">0.0</param>
+            <param name="p_lim_min">0.0</param>
+            <param name="p_offset">0.0</param>
+        </joint>
+        <joint name="LF_HFE"> <!-- hip -->
+            <param name="id">1</param>
+            <param name="bus">3</param>
+            <param name="motor_transmission">9.0</param> <!-- trasmissione primo motore link-->
+            <param name="sec_enc_transmission">0.0</param> <!-- trasmissione secondo motore2enc-->
+            <param name="KP">0.0</param>
+            <param name="KD">0.0</param>
+            <param name="KI">0.0</param>
+            <param name="i_limit">0.0</param>
+            <param name="p_lim_max">0.0</param>
+            <param name="p_lim_min">0.0</param>
+            <param name="p_offset">0.0</param>
+        </joint>
+        <joint name="LF_KFE"> <!-- hip -->
+            <param name="id">2</param>
+            <param name="bus">3</param>
+            <param name="motor_transmission">9.0</param> <!-- trasmissione primo motore link-->
+            <param name="sec_enc_transmission">0.0</param> <!-- trasmissione secondo motore2enc-->
+            <param name="KP">0.0</param>
+            <param name="KD">0.0</param>
+            <param name="KI">0.0</param>
+            <param name="i_limit">0.0</param>
+            <param name="p_lim_max">0.0</param>
+            <param name="p_lim_min">0.0</param>
+            <param name="p_offset">0.0</param>
+        </joint>
+        <joint name="LH_HFE"> <!-- hip -->
+            <param name="id">5</param>
+            <param name="bus">1</param>
+            <param name="motor_transmission">9.0</param> <!-- trasmissione primo motore link-->
+            <param name="sec_enc_transmission">0.0</param> <!-- trasmissione secondo motore2enc-->
+            <param name="KP">0.0</param>
+            <param name="KD">0.0</param>
+            <param name="KI">0.0</param>
+            <param name="i_limit">0.0</param>
+            <param name="p_lim_max">0.0</param>
+            <param name="p_lim_min">0.0</param>
+            <param name="p_offset">0.0</param>
+        </joint>
+        <joint name="LH_KFE"> <!-- hip -->
+            <param name="id">6</param>
+            <param name="bus">1</param>
+            <param name="motor_transmission">9.0</param> <!-- trasmissione primo motore link-->
+            <param name="sec_enc_transmission">0.0</param> <!-- trasmissione secondo motore2enc-->
+            <param name="KP">0.0</param>
+            <param name="KD">0.0</param>
+            <param name="KI">0.0</param>
+            <param name="i_limit">0.0</param>
+            <param name="p_lim_max">0.0</param>
+            <param name="p_lim_min">0.0</param>
+            <param name="p_offset">0.0</param>
+        </joint>
+        <joint name="RH_HFE"> <!-- hip -->
+            <param name="id">7</param>
+            <param name="bus">2</param>
+            <param name="motor_transmission">9.0</param> <!-- trasmissione primo motore link-->
+            <param name="sec_enc_transmission">0.0</param> <!-- trasmissione secondo motore2enc-->
+            <param name="KP">0.0</param>
+            <param name="KD">0.0</param>
+            <param name="KI">0.0</param>
+            <param name="i_limit">0.0</param>
+            <param name="p_lim_max">0.0</param>
+            <param name="p_lim_min">0.0</param>
+            <param name="p_offset">0.0</param>
+        </joint>
+        <joint name="RH_KFE"> <!-- hip -->
+            <!-- <param name="id">8</param> -->
+            <param name="bus">2</param>
+            <param name="motor_transmission">9.0</param> <!-- trasmissione primo motore link-->
+            <param name="sec_enc_transmission">0.0</param> <!-- trasmissione secondo motore2enc-->
+            <param name="KP">0.0</param>
+            <param name="KD">0.0</param>
+            <param name="KI">0.0</param>
+            <param name="i_limit">0.0</param>
+            <param name="p_lim_max">0.0</param>
+            <param name="p_lim_min">0.0</param>
+            <param name="p_offset">0.0</param>
+        </joint>
     </ros2_control>
 </robot>
