Commit message: tested joint limit and offset

File: pi3hat_hw_interface/urdf/test_int.urdf.xacro (robot description, xacro)
@@ -4,5 +4,5 @@
         <hardware>
             <plugin>pi3hat_hw_interface/MoteusPi3Hat_Interface</plugin>
-            <param name="main_timeout">400000</param>
+            <param name="main_timeout">800000</param>
             <param name="can_timeout">20000</param>
             <param name="rcv_timeout">20000</param>
@@ -25,97 +25,149 @@
             <param name="KI">0.0</param>
             <param name="i_limit">0.0</param>
-            <param name="p_lim_max">0.0</param>
-            <param name="p_lim_min">0.0</param>
+            <param name="p_lim_max">6.0</param>
+            <param name="p_lim_min">-6.0</param>
             <param name="p_offset">0.0</param>
         </joint>
-        <joint name="RF_KFE"> <!-- hip -->
+        <joint name="RF_KFE">
             <param name="id">4</param>
             <param name="bus">4</param>
-            <param name="motor_transmission">9.0</param> <!-- trasmissione primo motore link-->
-            <param name="sec_enc_transmission">0.0</param> <!-- trasmissione secondo motore2enc-->
+            <param name="motor_transmission">9.0</param>
+            <param name="sec_enc_transmission">0.0</param>
             <param name="KP">0.0</param>
             <param name="KD">0.0</param>
             <param name="KI">0.0</param>
             <param name="i_limit">0.0</param>
-            <param name="p_lim_max">0.0</param>
-            <param name="p_lim_min">0.0</param>
+            <param name="p_lim_max">6.0</param>
+            <param name="p_lim_min">-6.0</param>
             <param name="p_offset">0.0</param>
         </joint>
-        <joint name="LF_HFE"> <!-- hip -->
+        <joint name="LF_HFE">
             <param name="id">1</param>
             <param name="bus">3</param>
-            <param name="motor_transmission">9.0</param> <!-- trasmissione primo motore link-->
-            <param name="sec_enc_transmission">0.0</param> <!-- trasmissione secondo motore2enc-->
+            <param name="motor_transmission">9.0</param>
+            <param name="sec_enc_transmission">0.0</param>
             <param name="KP">0.0</param>
             <param name="KD">0.0</param>
             <param name="KI">0.0</param>
             <param name="i_limit">0.0</param>
-            <param name="p_lim_max">0.0</param>
-            <param name="p_lim_min">0.0</param>
+            <param name="p_lim_max">6.0</param>
+            <param name="p_lim_min">-6.0</param>
             <param name="p_offset">0.0</param>
         </joint>
-        <joint name="LF_KFE"> <!-- hip -->
+        <joint name="LF_KFE">
             <param name="id">2</param>
             <param name="bus">3</param>
-            <param name="motor_transmission">9.0</param> <!-- trasmissione primo motore link-->
-            <param name="sec_enc_transmission">0.0</param> <!-- trasmissione secondo motore2enc-->
+            <param name="motor_transmission">9.0</param>
+            <param name="sec_enc_transmission">0.0</param>
             <param name="KP">0.0</param>
             <param name="KD">0.0</param>
             <param name="KI">0.0</param>
             <param name="i_limit">0.0</param>
-            <param name="p_lim_max">0.0</param>
-            <param name="p_lim_min">0.0</param>
+            <param name="p_lim_max">6.0</param>
+            <param name="p_lim_min">-6.0</param>
             <param name="p_offset">0.0</param>
         </joint>
-        <joint name="LH_HFE"> <!-- hip -->
+        <joint name="LH_HFE">
             <param name="id">5</param>
             <param name="bus">1</param>
-            <param name="motor_transmission">9.0</param> <!-- trasmissione primo motore link-->
-            <param name="sec_enc_transmission">0.0</param> <!-- trasmissione secondo motore2enc-->
+            <param name="motor_transmission">9.0</param>
+            <param name="sec_enc_transmission">0.0</param>
             <param name="KP">0.0</param>
             <param name="KD">0.0</param>
             <param name="KI">0.0</param>
             <param name="i_limit">0.0</param>
-            <param name="p_lim_max">0.0</param>
-            <param name="p_lim_min">0.0</param>
+           <param name="p_lim_max">6.0</param>
+            <param name="p_lim_min">-6.0</param>
             <param name="p_offset">0.0</param>
         </joint>
-        <joint name="LH_KFE"> <!-- hip -->
+        <joint name="LH_KFE">
             <param name="id">6</param>
             <param name="bus">1</param>
-            <param name="motor_transmission">9.0</param> <!-- trasmissione primo motore link-->
-            <param name="sec_enc_transmission">0.0</param> <!-- trasmissione secondo motore2enc-->
+            <param name="motor_transmission">9.0</param>
+            <param name="sec_enc_transmission">0.0</param>
             <param name="KP">0.0</param>
             <param name="KD">0.0</param>
             <param name="KI">0.0</param>
             <param name="i_limit">0.0</param>
-            <param name="p_lim_max">0.0</param>
-            <param name="p_lim_min">0.0</param>
+            <param name="p_lim_max">6.0</param>
+            <param name="p_lim_min">-6.0</param>
             <param name="p_offset">0.0</param>
         </joint>
-        <joint name="RH_HFE"> <!-- hip -->
+        <joint name="RH_HFE">
             <param name="id">7</param>
             <param name="bus">2</param>
-            <param name="motor_transmission">9.0</param> <!-- trasmissione primo motore link-->
-            <param name="sec_enc_transmission">0.0</param> <!-- trasmissione secondo motore2enc-->
+            <param name="motor_transmission">9.0</param>
+            <param name="sec_enc_transmission">0.0</param>
             <param name="KP">0.0</param>
             <param name="KD">0.0</param>
             <param name="KI">0.0</param>
             <param name="i_limit">0.0</param>
-            <param name="p_lim_max">0.0</param>
-            <param name="p_lim_min">0.0</param>
+            <param name="p_lim_max">6.0</param>
+            <param name="p_lim_min">-6.0</param>
             <param name="p_offset">0.0</param>
         </joint>
-        <joint name="RH_KFE"> <!-- hip -->
-            <!-- <param name="id">8</param> -->
+        <joint name="RH_KFE">
+            <param name="id">8</param>
             <param name="bus">2</param>
-            <param name="motor_transmission">9.0</param> <!-- trasmissione primo motore link-->
-            <param name="sec_enc_transmission">0.0</param> <!-- trasmissione secondo motore2enc-->
+            <param name="motor_transmission">9.0</param>
+            <param name="sec_enc_transmission">0.0</param>
             <param name="KP">0.0</param>
             <param name="KD">0.0</param>
             <param name="KI">0.0</param>
             <param name="i_limit">0.0</param>
-            <param name="p_lim_max">0.0</param>
-            <param name="p_lim_min">0.0</param>
+            <param name="p_lim_max">6.0</param>
+            <param name="p_lim_min">-6.0</param>
+            <param name="p_offset">0.0</param>
+        </joint>
+        <joint name="RH_WHEEL">
+            <param name="id">12</param>
+            <param name="bus">2</param>
+            <param name="motor_transmission">15.0</param>
+            <param name="sec_enc_transmission">0.0</param>
+            <param name="KP">0.0</param>
+            <param name="KD">0.0</param>
+            <param name="KI">0.0</param>
+            <param name="i_limit">0.0</param>
+            <param name="p_lim_max">5000</param>
+            <param name="p_lim_min">-5000</param>
+            <param name="p_offset">0.0</param>
+        </joint>
+        <joint name="LH_WHEEL">
+            <param name="id">11</param>
+            <param name="bus">1</param>
+            <param name="motor_transmission">15.0</param>
+            <param name="sec_enc_transmission">0.0</param>
+            <param name="KP">0.0</param>
+            <param name="KD">0.0</param>
+            <param name="KI">0.0</param>
+            <param name="i_limit">0.0</param>
+            <param name="p_lim_max">5000</param>
+            <param name="p_lim_min">-5000</param>
+            <param name="p_offset">0.0</param>
+        </joint>
+        <joint name="LF_WHEEL">
+            <param name="id">9</param>
+            <param name="bus">3</param>
+            <param name="motor_transmission">15.0</param>
+            <param name="sec_enc_transmission">0.0</param>
+            <param name="KP">0.0</param>
+            <param name="KD">0.0</param>
+            <param name="KI">0.0</param>
+            <param name="i_limit">0.0</param>
+            <param name="p_lim_max">5000</param>
+            <param name="p_lim_min">-5000</param>
+            <param name="p_offset">0.0</param>
+        </joint>
+        <joint name="RF_WHEEL">
+            <param name="id">10</param>
+            <param name="bus">4</param>
+            <param name="motor_transmission">15.0</param>
+            <param name="sec_enc_transmission">0.0</param>
+            <param name="KP">0.0</param>
+            <param name="KD">0.0</param>
+            <param name="KI">0.0</param>
+            <param name="i_limit">0.0</param>
+            <param name="p_lim_max">5000</param>
+            <param name="p_lim_min">-5000</param>
             <param name="p_offset">0.0</param>
         </joint>

Commit message: fix imu corr

File: pi3hat_hw_interface/urdf/test_int.urdf.xacro (robot description, xacro)
@@ -7,5 +7,5 @@
             <param name="can_timeout">20000</param>
             <param name="rcv_timeout">20000</param>
-            <param name="attitude">1</param>
+            <param name="attitude">0</param>
             <param name="b2imu_pos_x">0</param>
             <param name="b2imu_pos_y">0</param>
@@ -16,5 +16,5 @@
             <param name="acc_correction">0</param>
         </hardware>
-        <joint name="RF_HFE">
+        <!-- <joint name="RF_HFE">
             <param name="id">3</param>
             <param name="bus">4</param>
@@ -171,5 +171,5 @@
             <param name="p_lim_min">-5000</param>
             <param name="p_offset">0.0</param>
-        </joint>
+        </joint> -->
     </ros2_control>
 </robot>
