Commit message: fix Gain conversion

File: pi3hat_hw_interface/urdf/test_ZERO.urdf.xacro (robot description, xacro)
@@ -7,5 +7,5 @@
             <param name="can_timeout">20000</param>
             <param name="rcv_timeout">20000</param>
-            <param name="attitude">0</param>
+            <param name="attitude">1</param>
             <param name="b2imu_pos_x">0</param>
             <param name="b2imu_pos_y">0</param>
@@ -14,13 +14,13 @@
             <param name="b2imu_pitch">0</param>
             <param name="b2imu_yaw">90.0</param>
-            <param name="acc_correction">1</param>
+            <param name="acc_correction">0</param>
         </hardware>
-        <joint name="RF_HFE">
+    	 <joint name="RF_HFE">
             <param name="id">3</param>
             <param name="bus">4</param>
             <param name="motor_transmission">9.0</param>
             <param name="sec_enc_transmission">0.0</param>
-            <param name="KP">70.9</param>
-            <param name="KD">0.4</param>
+            <param name="KP">0.0</param>
+            <param name="KD">0.0</param>
             <param name="KI">0.0</param>
             <param name="i_limit">0.0</param>
@@ -28,5 +28,5 @@
             <param name="p_lim_min">-3.14</param>
             <param name="p_offset">0.0</param>
-            <param name="max_vel">10.0</param>
+            <param name="max_vel">20.0</param>
         </joint>
         <joint name="RF_KFE">
@@ -35,6 +35,6 @@
             <param name="motor_transmission">9.0</param>
             <param name="sec_enc_transmission">0.0</param>
-            <param name="KP">70.9</param>
-            <param name="KD">0.4</param>
+            <param name="KP">0.0</param>
+            <param name="KD">0.0</param>
             <param name="KI">0.0</param>
             <param name="i_limit">0.0</param>
@@ -42,5 +42,5 @@
             <param name="p_lim_min">-3.14</param>
             <param name="p_offset">0.0</param>
-            <param name="max_vel">10.0</param>
+            <param name="max_vel">20.0</param>
         </joint>
         <joint name="LF_HFE">
@@ -49,6 +49,6 @@
             <param name="motor_transmission">9.0</param>
             <param name="sec_enc_transmission">0.0</param>
-            <param name="KP">70.9</param>
-            <param name="KD">0.4</param>
+            <param name="KP">0.0</param>
+            <param name="KD">0.0</param>
             <param name="KI">0.0</param>
             <param name="i_limit">0.0</param>
@@ -56,5 +56,5 @@
             <param name="p_lim_min">-3.14</param>
             <param name="p_offset">0.0</param>
-            <param name="max_vel">10.0</param>
+            <param name="max_vel">20.0</param>
         </joint>
         <joint name="LF_KFE">
@@ -63,6 +63,6 @@
             <param name="motor_transmission">9.0</param>
             <param name="sec_enc_transmission">0.0</param>
-            <param name="KP">70.9</param>
-            <param name="KD">0.4</param>
+            <param name="KP">0.0</param>
+            <param name="KD">0.0</param>
             <param name="KI">0.0</param>
             <param name="i_limit">0.0</param>
@@ -70,5 +70,5 @@
             <param name="p_lim_min">-3.14</param>
             <param name="p_offset">0.0</param>
-            <param name="max_vel">10.0</param>
+            <param name="max_vel">20.0</param>
         </joint>
         <joint name="LH_HFE">
@@ -77,6 +77,6 @@
             <param name="motor_transmission">9.0</param>
             <param name="sec_enc_transmission">0.0</param>
-            <param name="KP">70.9</param>
-            <param name="KD">0.4</param>
+            <param name="KP">0.0</param>
+            <param name="KD">0.0</param>
             <param name="KI">0.0</param>
             <param name="i_limit">0.0</param>
@@ -84,5 +84,5 @@
             <param name="p_lim_min">-3.14</param>
             <param name="p_offset">0.0</param>
-            <param name="max_vel">10.0</param>
+            <param name="max_vel">20.0</param>
         </joint>
         <joint name="LH_KFE">
@@ -91,6 +91,6 @@
             <param name="motor_transmission">9.0</param>
             <param name="sec_enc_transmission">0.0</param>
-            <param name="KP">70.9</param>
-            <param name="KD">0.4</param>
+            <param name="KP">0.0</param>
+            <param name="KD">0.0</param>
             <param name="KI">0.0</param>
             <param name="i_limit">0.0</param>
@@ -98,5 +98,5 @@
             <param name="p_lim_min">-3.14</param>
             <param name="p_offset">0.0</param>
-            <param name="max_vel">10.0</param>
+            <param name="max_vel">20.0</param>
         </joint>
         <joint name="RH_HFE">
@@ -105,6 +105,6 @@
             <param name="motor_transmission">9.0</param>
             <param name="sec_enc_transmission">0.0</param>
-            <param name="KP">70.9</param>
-            <param name="KD">0.4</param>
+            <param name="KP">0.0</param>
+            <param name="KD">0.0</param>
             <param name="KI">0.0</param>
             <param name="i_limit">0.0</param>
@@ -112,5 +112,5 @@
             <param name="p_lim_min">-3.14</param>
             <param name="p_offset">0.0</param>
-            <param name="max_vel">10.0</param>
+            <param name="max_vel">20.0</param>
         </joint>
         <joint name="RH_KFE">
@@ -119,6 +119,6 @@
             <param name="motor_transmission">9.0</param>
             <param name="sec_enc_transmission">0.0</param>
-            <param name="KP">70.9</param>
-            <param name="KD">0.4</param>
+            <param name="KP">0.0</param>
+            <param name="KD">0.0</param>
             <param name="KI">0.0</param>
             <param name="i_limit">0.0</param>
@@ -126,18 +126,19 @@
             <param name="p_lim_min">-3.14</param>
             <param name="p_offset">0.0</param>
-            <param name="max_vel">10.0</param>
+            <param name="max_vel">20.0</param>
         </joint>
-       <!-- <joint name="RH_WHEEL">
+       <!--  <joint name="RH_WHEEL">
             <param name="id">12</param>
             <param name="bus">2</param>
             <param name="motor_transmission">15.0</param>
             <param name="sec_enc_transmission">0.0</param>
-            <param name="KP">0.0</param>
-            <param name="KD">0.0</param>
+            <param name="KP">5.0</param>
+            <param name="KD">0.025</param>
             <param name="KI">0.0</param>
             <param name="i_limit">0.0</param>
-            <param name="p_lim_max">5000</param>
-            <param name="p_lim_min">-5000</param>
+            <param name="p_lim_max">0.0</param>
+            <param name="p_lim_min">0.0</param>
             <param name="p_offset">0.0</param>
+            <param name="max_vel">50.0</param>
         </joint>
         <joint name="LH_WHEEL">
@@ -150,20 +151,22 @@
             <param name="KI">0.0</param>
             <param name="i_limit">0.0</param>
-            <param name="p_lim_max">5000</param>
-            <param name="p_lim_min">-5000</param>
+            <param name="p_lim_max">0.0</param>
+            <param name="p_lim_min">0.0</param>
             <param name="p_offset">0.0</param>
+            <param name="max_vel">50.0</param>
         </joint>
-        <joint name="LF_WHEEL">
+         <joint name="LF_WHEEL">
             <param name="id">9</param>
             <param name="bus">3</param>
             <param name="motor_transmission">15.0</param>
             <param name="sec_enc_transmission">0.0</param>
-            <param name="KP">0.0</param>
-            <param name="KD">0.0</param>
+            <param name="KP">5.0</param>
+            <param name="KD">0.025</param>
             <param name="KI">0.0</param>
             <param name="i_limit">0.0</param>
-            <param name="p_lim_max">5000</param>
-            <param name="p_lim_min">-5000</param>
+            <param name="p_lim_max">0.0</param>
+            <param name="p_lim_min">0.0</param>
             <param name="p_offset">0.0</param>
+            <param name="max_vel">50.0</param>
         </joint>
         <joint name="RF_WHEEL">
@@ -172,12 +175,13 @@
             <param name="motor_transmission">15.0</param>
             <param name="sec_enc_transmission">0.0</param>
-            <param name="KP">0.0</param>
-            <param name="KD">0.0</param>
+            <param name="KP">5.0</param>
+            <param name="KD">0.025</param>
             <param name="KI">0.0</param>
             <param name="i_limit">0.0</param>
-            <param name="p_lim_max">5000</param>
-            <param name="p_lim_min">-5000</param>
+            <param name="p_lim_max">0.0</param>
+            <param name="p_lim_min">0.0</param>
             <param name="p_offset">0.0</param>
-        </joint>-->
+            <param name="max_vel">50.0</param>
+        </joint> -->
     </ros2_control>
 </robot>
