Commit message: bench launch and test launch

File: pi3hat_hw_interface/urdf/8DOF_mul_RLTESTS.urdf.xacro (robot description, xacro)
@@ -4,8 +4,8 @@
         <hardware>
             <plugin>pi3hat_hw_interface/MoteusPi3Hat_Interface</plugin>
-            <param name="main_timeout">1000000</param>
-            <param name="can_timeout">40000</param>
-            <param name="rcv_timeout">40000</param>
-            <param name="attitude">0</param>
+            <param name="main_timeout">800000</param>
+            <param name="can_timeout">20000</param>
+            <param name="rcv_timeout">20000</param>
+            <param name="attitude">1</param>
             <param name="b2imu_pos_x">0</param>
             <param name="b2imu_pos_y">0</param>
@@ -26,6 +26,6 @@
             <param name="max_torque">6.0</param>
             -->
-	        <param name="KP">200</param>
-            <param name="KD">0.95</param>
+	        <param name="KP">30.0</param>
+            <param name="KD">0.14</param>
             <param name="KI">0.0</param>
             <param name="i_limit">0.0</param>
@@ -34,5 +34,5 @@
             <param name="p_offset">0.0</param>
             <param name="max_vel">10.0</param>
-            <param name="max_torque">15.0</param>
+            <param name="max_torque">5.0</param>
         </joint>
         <joint name="RF_KFE">
@@ -41,6 +41,6 @@
             <param name="motor_transmission">9.0</param>
             <param name="sec_enc_transmission">0.0</param>
-            <param name="KP">200</param>
-            <param name="KD">0.95</param>
+            <param name="KP">30.0</param>
+            <param name="KD">0.14</param>
             <param name="KI">0.0</param>
             <param name="i_limit">0.0</param>
@@ -49,5 +49,5 @@
             <param name="p_offset">-0.1059179</param>
             <param name="max_vel">10.0</param>
-            <param name="max_torque">15.0</param>
+            <param name="max_torque">5.0</param>
         </joint>
         <joint name="LF_HFE">
@@ -56,6 +56,6 @@
             <param name="motor_transmission">9.0</param>
             <param name="sec_enc_transmission">0.0</param>
-            <param name="KP">200</param>
-            <param name="KD">0.95</param>
+            <param name="KP">30.0</param>
+            <param name="KD">0.14</param>
             <param name="KI">0.0</param>
             <param name="i_limit">0.0</param>
@@ -64,5 +64,5 @@
             <param name="p_offset">0.0</param>
             <param name="max_vel">10.0</param>
-            <param name="max_torque">15.0</param>
+            <param name="max_torque">5.0</param>
         </joint>
         <joint name="LF_KFE">
@@ -71,6 +71,6 @@
             <param name="motor_transmission">9.0</param>
             <param name="sec_enc_transmission">0.0</param>
-            <param name="KP">200</param>
-            <param name="KD">0.95</param>
+            <param name="KP">30.0</param>
+            <param name="KD">0.14</param>
             <param name="KI">0.0</param>
             <param name="i_limit">0.0</param>
@@ -79,5 +79,5 @@
             <param name="p_offset">0.1059179</param>
             <param name="max_vel">10.0</param>
-            <param name="max_torque">15.0</param>
+            <param name="max_torque">5.0</param>
         </joint>
         <joint name="LH_HFE">
@@ -86,6 +86,6 @@
             <param name="motor_transmission">9.0</param>
             <param name="sec_enc_transmission">0.0</param>
-            <param name="KP">200</param>
-            <param name="KD">0.95</param>
+            <param name="KP">30.0</param>
+            <param name="KD">0.14</param>
             <param name="KI">0.0</param>
             <param name="i_limit">0.0</param>
@@ -94,5 +94,5 @@
             <param name="p_offset">0.0</param>
             <param name="max_vel">10.0</param>
-            <param name="max_torque">15.0</param>
+            <param name="max_torque">5.0</param>
         </joint>
         <joint name="LH_KFE">
@@ -101,6 +101,6 @@
             <param name="motor_transmission">9.0</param>
             <param name="sec_enc_transmission">0.0</param>
-            <param name="KP">200</param>
-            <param name="KD">0.95</param>
+            <param name="KP">30.0</param>
+            <param name="KD">0.14</param>
             <param name="KI">0.0</param>
             <param name="i_limit">0.0</param>
@@ -109,5 +109,5 @@
             <param name="p_offset">-0.1059179</param>
             <param name="max_vel">10.0</param>
-            <param name="max_torque">15.0</param>
+            <param name="max_torque">5.0</param>
         </joint>
         <joint name="RH_HFE">
@@ -116,6 +116,6 @@
             <param name="motor_transmission">9.0</param>
             <param name="sec_enc_transmission">0.0</param>
-            <param name="KP">200</param>
-            <param name="KD">0.95</param>
+            <param name="KP">30.0</param>
+            <param name="KD">0.14</param>
             <param name="KI">0.0</param>
             <param name="i_limit">0.0</param>
@@ -124,5 +124,5 @@
             <param name="p_offset">0.0</param>
             <param name="max_vel">10.0</param>
-            <param name="max_torque">15.0</param>
+            <param name="max_torque">5.0</param>
         </joint>
         <joint name="RH_KFE">
@@ -131,6 +131,6 @@
             <param name="motor_transmission">9.0</param>
             <param name="sec_enc_transmission">0.0</param>
-            <param name="KP">200</param>
-            <param name="KD">0.95</param>
+            <param name="KP">30.0</param>
+            <param name="KD">0.14</param>
             <param name="KI">0.0</param>
             <param name="i_limit">0.0</param>
@@ -139,5 +139,5 @@
             <param name="p_offset">0.1059179</param>
             <param name="max_vel">10.0</param>
-            <param name="max_torque">15.0</param>
+            <param name="max_torque">5.0</param>
         </joint>
     </ros2_control>

File: pi3hat_hw_interface/urdf/ILC_8DOF_mul_off.urdf.xacro (robot description, xacro)
@@ -4,7 +4,7 @@
         <hardware>
             <plugin>pi3hat_hw_interface/MoteusPi3Hat_Interface</plugin>
-            <param name="main_timeout">1000000</param>
-            <param name="can_timeout">40000</param>
-            <param name="rcv_timeout">40000</param>
+            <param name="main_timeout">800000</param>
+            <param name="can_timeout">20000</param>
+            <param name="rcv_timeout">20000</param>
             <param name="attitude">0</param>
             <param name="b2imu_pos_x">0</param>
@@ -26,6 +26,6 @@
             <param name="max_torque">6.0</param>
             -->
-	        <param name="KP">200</param>
-            <param name="KD">0.95</param>
+	        <param name="KP">320</param>
+            <param name="KD">1.0</param>
             <param name="KI">0.0</param>
             <param name="i_limit">0.0</param>
@@ -41,6 +41,6 @@
             <param name="motor_transmission">9.0</param>
             <param name="sec_enc_transmission">0.0</param>
-            <param name="KP">200</param>
-            <param name="KD">0.95</param>
+            <param name="KP">320</param>
+            <param name="KD">1.0</param>
             <param name="KI">0.0</param>
             <param name="i_limit">0.0</param>
@@ -56,6 +56,6 @@
             <param name="motor_transmission">9.0</param>
             <param name="sec_enc_transmission">0.0</param>
-            <param name="KP">200</param>
-            <param name="KD">0.95</param>
+            <param name="KP">320</param>
+            <param name="KD">1.0</param>
             <param name="KI">0.0</param>
             <param name="i_limit">0.0</param>
@@ -71,6 +71,6 @@
             <param name="motor_transmission">9.0</param>
             <param name="sec_enc_transmission">0.0</param>
-            <param name="KP">200</param>
-            <param name="KD">0.95</param>
+            <param name="KP">320</param>
+            <param name="KD">1.0</param>
             <param name="KI">0.0</param>
             <param name="i_limit">0.0</param>
@@ -86,6 +86,6 @@
             <param name="motor_transmission">9.0</param>
             <param name="sec_enc_transmission">0.0</param>
-            <param name="KP">200</param>
-            <param name="KD">0.95</param>
+            <param name="KP">320</param>
+            <param name="KD">1.0</param>
             <param name="KI">0.0</param>
             <param name="i_limit">0.0</param>
@@ -101,6 +101,6 @@
             <param name="motor_transmission">9.0</param>
             <param name="sec_enc_transmission">0.0</param>
-            <param name="KP">200</param>
-            <param name="KD">0.95</param>
+            <param name="KP">320</param>
+            <param name="KD">1.0</param>
             <param name="KI">0.0</param>
             <param name="i_limit">0.0</param>
@@ -116,6 +116,6 @@
             <param name="motor_transmission">9.0</param>
             <param name="sec_enc_transmission">0.0</param>
-            <param name="KP">200</param>
-            <param name="KD">0.95</param>
+            <param name="KP">320</param>
+            <param name="KD">1.0</param>
             <param name="KI">0.0</param>
             <param name="i_limit">0.0</param>
@@ -131,6 +131,6 @@
             <param name="motor_transmission">9.0</param>
             <param name="sec_enc_transmission">0.0</param>
-            <param name="KP">200</param>
-            <param name="KD">0.95</param>
+            <param name="KP">320</param>
+            <param name="KD">1.0</param>
             <param name="KI">0.0</param>
             <param name="i_limit">0.0</param>

File: pi3hat_hw_interface/urdf/bench_test.urdf.xacro (robot description, xacro)
@@ -20,4 +20,129 @@
             <param name="acc_correction">1</param>
         </hardware>
+                <joint name="RF_HFE">
+            <param name="id">3</param>
+            <param name="bus">4</param>
+            <param name="motor_transmission">9.0</param>
+            <param name="sec_enc_transmission">0.0</param>
+            <!-- JOSH PARAM
+            <param name="KP">15</param>
+            <param name="KD">0.1</param>
+            <param name="max_torque">6.0</param>
+            -->
+	    <param name="KP">70.9</param>
+            <param name="KD">0.4</param>
+            <param name="KI">0.0</param>
+            <param name="i_limit">0.0</param>
+            <param name="p_lim_max">3.14</param>
+            <param name="p_lim_min">-3.14</param>
+            <param name="p_offset">0.0</param>
+            <param name="max_vel">10.0</param>
+            <param name="max_torque">5.0</param>
+        </joint>
+        <joint name="RF_KFE">
+            <param name="id">4</param>
+            <param name="bus">4</param>
+            <param name="motor_transmission">9.0</param>
+            <param name="sec_enc_transmission">0.0</param>
+            <param name="KP">70.9</param>
+            <param name="KD">0.4</param>
+            <param name="KI">0.0</param>
+            <param name="i_limit">0.0</param>
+            <param name="p_lim_max">3.14</param>
+            <param name="p_lim_min">-3.14</param>
+            <param name="p_offset">-0.1059179</param>
+            <param name="max_vel">10.0</param>
+            <param name="max_torque">5.0</param>
+        </joint>
+        <joint name="LF_HFE">
+            <param name="id">1</param>
+            <param name="bus">3</param>
+            <param name="motor_transmission">9.0</param>
+            <param name="sec_enc_transmission">0.0</param>
+            <param name="KP">70.9</param>
+            <param name="KD">0.4</param>
+            <param name="KI">0.0</param>
+            <param name="i_limit">0.0</param>
+            <param name="p_lim_max">3.14</param>
+            <param name="p_lim_min">-3.14</param>
+            <param name="p_offset">0.0</param>
+            <param name="max_vel">10.0</param>
+            <param name="max_torque">5.0</param>
+        </joint>
+        <joint name="LF_KFE">
+            <param name="id">2</param>
+            <param name="bus">3</param>
+            <param name="motor_transmission">9.0</param>
+            <param name="sec_enc_transmission">0.0</param>
+            <param name="KP">70.9</param>
+            <param name="KD">0.4</param>
+            <param name="KI">0.0</param>
+            <param name="i_limit">0.0</param>
+            <param name="p_lim_max">3.14</param>
+            <param name="p_lim_min">-3.14</param>
+            <param name="p_offset">0.1059179</param>
+            <param name="max_vel">10.0</param>
+            <param name="max_torque">5.0</param>
+        </joint>
+        <joint name="LH_HFE">
+            <param name="id">5</param>
+            <param name="bus">1</param>
+            <param name="motor_transmission">9.0</param>
+            <param name="sec_enc_transmission">0.0</param>
+            <param name="KP">70.9</param>
+            <param name="KD">0.4</param>
+            <param name="KI">0.0</param>
+            <param name="i_limit">0.0</param>
+           <param name="p_lim_max">3.14</param>
+            <param name="p_lim_min">-3.14</param>
+            <param name="p_offset">0.0</param>
+            <param name="max_vel">10.0</param>
+            <param name="max_torque">5.0</param>
+        </joint>
+        <joint name="LH_KFE">
+            <param name="id">6</param>
+            <param name="bus">1</param>
+            <param name="motor_transmission">9.0</param>
+            <param name="sec_enc_transmission">0.0</param>
+            <param name="KP">70.9</param>
+            <param name="KD">0.4</param>
+            <param name="KI">0.0</param>
+            <param name="i_limit">0.0</param>
+            <param name="p_lim_max">3.14</param>
+            <param name="p_lim_min">-3.14</param>
+            <param name="p_offset">-0.1059179</param>
+            <param name="max_vel">10.0</param>
+            <param name="max_torque">5.0</param>
+        </joint>
+        <joint name="RH_HFE">
+            <param name="id">7</param>
+            <param name="bus">2</param>
+            <param name="motor_transmission">9.0</param>
+            <param name="sec_enc_transmission">0.0</param>
+            <param name="KP">70.9</param>
+            <param name="KD">0.4</param>
+            <param name="KI">0.0</param>
+            <param name="i_limit">0.0</param>
+            <param name="p_lim_max">3.14</param>
+            <param name="p_lim_min">-3.14</param>
+            <param name="p_offset">0.0</param>
+            <param name="max_vel">10.0</param>
+            <param name="max_torque">5.0</param>
+        </joint>
+        <joint name="RH_KFE">
+            <param name="id">8</param>
+            <param name="bus">2</param>
+            <param name="motor_transmission">9.0</param>
+            <param name="sec_enc_transmission">0.0</param>
+            <param name="KP">70.9</param>
+            <param name="KD">0.4</param>
+            <param name="KI">0.0</param>
+            <param name="i_limit">0.0</param>
+            <param name="p_lim_max">3.14</param>
+            <param name="p_lim_min">-3.14</param>
+            <param name="p_offset">0.1059179</param>
+            <param name="max_vel">10.0</param>
+            <param name="max_torque">5.0</param>
+        </joint>
     </ros2_control>
 </robot>
