Commit message: add omnicar controller

File: pi3hat_hw_interface/urdf/bench_test.urdf.xacro (robot description, xacro)
@@ -20,25 +20,65 @@
             <param name="acc_correction">1</param>
         </hardware>
-                <joint name="RF_HFE">
-            <param name="id">3</param>
+        <joint name="RF_WHEEL">
+            <param name="id">2</param>
             <param name="bus">4</param>
             <param name="motor_transmission">9.0</param>
             <param name="sec_enc_transmission">0.0</param>
-            <!-- JOSH PARAM
-            <param name="KP">15</param>
-            <param name="KD">0.1</param>
-            <param name="max_torque">6.0</param>
-            -->
-	    <param name="KP">70.9</param>
-            <param name="KD">0.4</param>
+            <param name="KP">20</param>
+            <param name="KD">0.95</param>
             <param name="KI">0.0</param>
             <param name="i_limit">0.0</param>
-            <param name="p_lim_max">3.14</param>
-            <param name="p_lim_min">-3.14</param>
+            <param name="p_lim_max">900</param>
+            <param name="p_lim_min">-900</param>
+            <param name="p_offset">-0.1059179</param>
+            <param name="max_vel">100.0</param>
+            <param name="max_torque">15.0</param>
+        </joint>
+        <joint name="LF_WHEEL">
+            <param name="id">1</param>
+            <param name="bus">3</param>
+            <param name="motor_transmission">9.0</param>
+            <param name="sec_enc_transmission">0.0</param>
+            <param name="KP">20</param>
+            <param name="KD">0.95</param>
+            <param name="KI">0.0</param>
+            <param name="i_limit">0.0</param>
+            <param name="p_lim_max">900</param>
+            <param name="p_lim_min">-900</param>
             <param name="p_offset">0.0</param>
-            <param name="max_vel">10.0</param>
-            <param name="max_torque">5.0</param>
+            <param name="max_vel">100.0</param>
+            <param name="max_torque">15.0</param>
         </joint>
-        <joint name="RF_KFE">
+        <joint name="RH_WHEEL">
+            <param name="id">3</param>
+            <param name="bus">2</param>
+            <param name="motor_transmission">9.0</param>
+            <param name="sec_enc_transmission">0.0</param>
+            <param name="KP">20</param>
+            <param name="KD">0.95</param>
+            <param name="KI">0.0</param>
+            <param name="i_limit">0.0</param>
+            <param name="p_lim_max">900</param>
+            <param name="p_lim_min">-900</param>
+            <param name="p_offset">0.1059179</param>
+            <param name="max_vel">100.0</param>
+            <param name="max_torque">15.0</param>
+        </joint>
+         <joint name="LH_WHEEL">
+            <param name="id">4</param>
+            <param name="bus">1</param>
+            <param name="motor_transmission">9.0</param>
+            <param name="sec_enc_transmission">0.0</param>
+	        <param name="KP">20</param>
+            <param name="KD">0.95</param>
+            <param name="KI">0.0</param>
+            <param name="i_limit">0.0</param>
+            <param name="p_lim_max">900</param>
+            <param name="p_lim_min">-900</param>
+            <param name="p_offset">0.0</param>
+            <param name="max_vel">100.0</param>
+            <param name="max_torque">15.0</param>
+        </joint>
+        <!-- <joint name="RF_KFE">
             <param name="id">4</param>
             <param name="bus">4</param>
@@ -144,5 +184,5 @@
             <param name="max_vel">10.0</param>
             <param name="max_torque">5.0</param>
-        </joint>
+        </joint> -->
     </ros2_control>
 </robot>

Commit message: fix omni odometry and update readme

File: pi3hat_hw_interface/urdf/bench_test.urdf.xacro (robot description, xacro)
@@ -80,109 +80,4 @@
             <param name="max_torque">15.0</param>
         </joint>
-        <!-- <joint name="RF_KFE">
-            <param name="id">4</param>
-            <param name="bus">4</param>
-            <param name="motor_transmission">9.0</param>
-            <param name="sec_enc_transmission">0.0</param>
-            <param name="KP">70.9</param>
-            <param name="KD">0.4</param>
-            <param name="KI">0.0</param>
-            <param name="i_limit">0.0</param>
-            <param name="p_lim_max">3.14</param>
-            <param name="p_lim_min">-3.14</param>
-            <param name="p_offset">-0.1059179</param>
-            <param name="max_vel">10.0</param>
-            <param name="max_torque">5.0</param>
-        </joint>
-        <joint name="LF_HFE">
-            <param name="id">1</param>
-            <param name="bus">3</param>
-            <param name="motor_transmission">9.0</param>
-            <param name="sec_enc_transmission">0.0</param>
-            <param name="KP">70.9</param>
-            <param name="KD">0.4</param>
-            <param name="KI">0.0</param>
-            <param name="i_limit">0.0</param>
-            <param name="p_lim_max">3.14</param>
-            <param name="p_lim_min">-3.14</param>
-            <param name="p_offset">0.0</param>
-            <param name="max_vel">10.0</param>
-            <param name="max_torque">5.0</param>
-        </joint>
-        <joint name="LF_KFE">
-            <param name="id">2</param>
-            <param name="bus">3</param>
-            <param name="motor_transmission">9.0</param>
-            <param name="sec_enc_transmission">0.0</param>
-            <param name="KP">70.9</param>
-            <param name="KD">0.4</param>
-            <param name="KI">0.0</param>
-            <param name="i_limit">0.0</param>
-            <param name="p_lim_max">3.14</param>
-            <param name="p_lim_min">-3.14</param>
-            <param name="p_offset">0.1059179</param>
-            <param name="max_vel">10.0</param>
-            <param name="max_torque">5.0</param>
-        </joint>
-        <joint name="LH_HFE">
-            <param name="id">5</param>
-            <param name="bus">1</param>
-            <param name="motor_transmission">9.0</param>
-            <param name="sec_enc_transmission">0.0</param>
-            <param name="KP">70.9</param>
-            <param name="KD">0.4</param>
-            <param name="KI">0.0</param>
-            <param name="i_limit">0.0</param>
-           <param name="p_lim_max">3.14</param>
-            <param name="p_lim_min">-3.14</param>
-            <param name="p_offset">0.0</param>
-            <param name="max_vel">10.0</param>
-            <param name="max_torque">5.0</param>
-        </joint>
-        <joint name="LH_KFE">
-            <param name="id">6</param>
-            <param name="bus">1</param>
-            <param name="motor_transmission">9.0</param>
-            <param name="sec_enc_transmission">0.0</param>
-            <param name="KP">70.9</param>
-            <param name="KD">0.4</param>
-            <param name="KI">0.0</param>
-            <param name="i_limit">0.0</param>
-            <param name="p_lim_max">3.14</param>
-            <param name="p_lim_min">-3.14</param>
-            <param name="p_offset">-0.1059179</param>
-            <param name="max_vel">10.0</param>
-            <param name="max_torque">5.0</param>
-        </joint>
-        <joint name="RH_HFE">
-            <param name="id">7</param>
-            <param name="bus">2</param>
-            <param name="motor_transmission">9.0</param>
-            <param name="sec_enc_transmission">0.0</param>
-            <param name="KP">70.9</param>
-            <param name="KD">0.4</param>
-            <param name="KI">0.0</param>
-            <param name="i_limit">0.0</param>
-            <param name="p_lim_max">3.14</param>
-            <param name="p_lim_min">-3.14</param>
-            <param name="p_offset">0.0</param>
-            <param name="max_vel">10.0</param>
-            <param name="max_torque">5.0</param>
-        </joint>
-        <joint name="RH_KFE">
-            <param name="id">8</param>
-            <param name="bus">2</param>
-            <param name="motor_transmission">9.0</param>
-            <param name="sec_enc_transmission">0.0</param>
-            <param name="KP">70.9</param>
-            <param name="KD">0.4</param>
-            <param name="KI">0.0</param>
-            <param name="i_limit">0.0</param>
-            <param name="p_lim_max">3.14</param>
-            <param name="p_lim_min">-3.14</param>
-            <param name="p_offset">0.1059179</param>
-            <param name="max_vel">10.0</param>
-            <param name="max_torque">5.0</param>
-        </joint> -->
     </ros2_control>
 </robot>
